File: Hardware/MEchaduino_03.sch (EAGLE design)
At the start: 45 parts, among them Q2 NFET, U1 TLV70233PDBVR, U2 ATSAMD51G-M, U3 TXB0104, Y2 32,768Khz

Commit message: changed microcontroller to ATSAMD51J19
Parts:
- removed Q2: NFET, SparkFun-DiscreteSemi:MOSFET-NCHANNEL2N7002PW
- removed R4: 100k, rcl:R-US_R0402
- removed U$3: TROPICAL_LABS_LOGO_1LOGO3, stepper_servo_prototype_1:TROPICAL_LABS_LOGO_1LOGO3
- added C15, C18, C20, C21, C22: 0.1uF, swift:CAP0402
- added R6: 10k, rcl:R-US_R0402
- added SJ1: (no value), jumper:SJ
- C17, C3: value 18pF -> 22pF
- R1: value 330 -> 1k
- U2: value ATSAMD51G-M -> ATSAMD51J19; device atsamd51:ATSAMD51G-M -> atsamd51:ATSAMD51J19
Connections:
- removed net ARDUINO_D13_SCK: Q2.G, R4.2
- removed net GND2: J2.1
- removed net HEADER_MISO: U$4.MISO, U2.PA14(XIN/SER2:2+)
- removed net HEADER_MOSI: U$4.MOSI, U2.PA12(I2C/SER2:0+)
- removed net HEADER_SCK: U$4.CLK, U2.PA13(I2C/SER2:1+)
- removed net HEADER_SS: U$4.CSN, U2.PA06(AIN6/SER0:2/TC1:0)
- removed net N$11: J3.PIN3, U3.B4
- removed net N$12: J3.PIN2, U3.B3
- removed net N$17: J3.PIN1, U3.B2
- removed net N$18: J3.PIN0, U3.B1
- removed net N$3: Q2.D, R1.1
- removed net PA00_XIN1: C3.2, U2.PA00(XIN32/SER1:0/TC2:0), Y2.2
- removed net PA01_XOUT1: C17.2, U2.PA01(XOUT32/SER1:1/TC2:1), Y2.1
- removed net SCL: U2.PB03(AIN15/SER5:1)
- removed net SDA: U2.PB02(AIN14/SER5:0)
- removed net TARGET_USB_N: J1.D-, U2.PA24(USB/DM/SER3:2+)
- removed net TARGET_USB_P: J1.D+, U2.PA25(USB/DP/SER3:3+)
- removed net VDDANA: C5.1, L2.2, U2.VDDANA
- new net AREF: C22.1, SJ1.2, U2.PA03/I3/VREF/AIN1
- new net CRYST1: C3.2, U2.PA00/EINT0/SERCOM1.0, Y2.2
- new net CRYST2: C17.2, U2.PA01/EINT1/SERCOM1.1, Y2.1
- new net D+: J1.D+, U2.PA25/19/SERCOM3+5.3/D+
- new net D-: J1.D-, U2.PA24/I8/SERCOM3+5.2/D-
- new net D13: R1.2, U2.PA16/I2C/I0/SERCOM1.0+3.1
- new net MISO: U$4.MISO, U2.PA14/I14/SEROM2+4.2
- new net MOSI: U$4.MOSI, U2.PA12/I12/I2C/SEROM2.0+4.1
- new net N$10: L2.2, U2.VSW
- new net N$2: J3.PIN3, U3.B1
- new net N$4: J3.PIN2, U3.B2
- new net SCK: U$4.CLK, U2.PA13/I13/I2C/SEROM2.1+4.0
- new net SS: U$4.CSN, U2.PA15/I15/SEROM2+4.3
- net 3.3V: now also C10.1, C11.2, C14.1, C18.1, C20.1, R6.1, SJ1.1, U2.VDDANA, U2.VDDIO@21, U2.VDDIO@34, U2.VDDIO@48, U2.VDDIO@56; no longer C1.1, L2.1, LED1.A, U2.PA03(AIN1/REFA), U2.PA04(AIN4/REFB/SER0:0/TC0:0), U2.VDDIN
- net A: now also U2.PB14/I14/SERCOM4.2/PCC8; no longer U2.PA08(I2S/AIN8/SER0:0+)
- net ARDUINO_D0: now also U2.PA23/I2C/I7/SERCOM3.1+5.0/SOF/I2SFS1, U3.A1; no longer U2.PA16(I2C/SER1:0+), U3.A4
- net ARDUINO_D1: now also U2.PA22/I2C/16/SERCOM3.0+5.1/I2SFS1, U3.A2; no longer U2.PA17(I2C/SER1:1+), U3.A3
- net ARDUINO_D2: now also U2.PB17/SERCOM5.1/I2SMCK0, U3.A3; no longer U2.PA18(SER1:2+), U3.A2
- net ARDUINO_D3: now also U2.PB16/I0/SERCOM5.0/I2SCK0, U3.A4; no longer U2.PA19(SER1:3+), U3.A1
- net B: now also U2.PB13/I13/SERCOM4.1/I2SMCK1; no longer U2.PA09(I2S/AIN9/SER0:1+)
- net GND: now also C15.1, C18.2, C20.2, C21.2, C22.2, J2.1, LED1.C, SW2.P$4, U2.GND@22, U2.GND@33, U2.GND@47, U2.GND@54, U2.GND@7; no longer C11.2, Q2.S, R4.1, U2.GND@18, U2.GND@35, U2.GND@42, U2.GND@5
- net I: now also U2.PB15/I15/SERCOM4.3/PCC9; no longer U2.PA10(AIN10/SER0:2+)
- net IN1: now also U2.PA18/I2/SEROM1+3.2; no longer U2.PA20(I2S/SER5:2+)
- net IN2: now also U2.PA19/I3/SEROM1+3.3; no longer U2.PA21(I2S/SER5:3+)
- net IN3: now also U2.PA21/I5/SERCOM3+5.3/I2SDO; no longer U2.PA23(I2C/SER3:0+)
- net IN4: now also U2.PA20/I4/SERCOM3/5.2/I2SFS0; no longer U2.PA22(I2C/SER3:0+)
- net N$1: now also LED1.A, R1.1; no longer LED1.C, R1.2
- net N$5: now also J3.PIN1, U3.B3; no longer C14.1, U2.VDDIO@36
- net N$7: now also J3.PIN0, U3.B4; no longer C10.1, U2.VDDIO@17
- net N$8: now also C1.1, C21.1, C5.1, L2.1
- net RESET: now also C15.2, R6.2, SW2.P$2
- net TH1: now also U2.PA07/I7/AIN7/SERCOM0.3; no longer U2.PB09(AIN3/SER4:1/TC4:1)
- net VREF1: now also U2.PA05/I5/AIN5/VOUT1/SERCOM0.1; no longer U2.PA05(AIN5/VOUT2/SER0:1/TC0:1)
- net VREF2: now also U2.PA02/EINT2/AIN0/VOUT0; no longer U2.PA02(AIN0/VOUT0)
Other:
- moved on the sheet: C1, C10, C11, C14, C17, C2, C3, C5, J3, L2, LED1, R1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

Commit message: implemted voltage sense pin and some leds
Parts:
- removed F1: 500mA, SparkFun-PowerIC:PTCSMD
- added F2: 500mA, adafruit:PTCFUSE-1206
- added LED2: Red, Opto:0044_KPT-2012YC
- added LED3: Green, Opto:0044_KPT-2012YC
- added R4: 100k, rcl:R-US_R0402
- added R7: 6k8, rcl:R-US_R0402
- added R8, R9: 1k, rcl:R-US_R0402
- J1: value (none) -> USB
- J2: value (none) -> power
- J3: value (none) -> signals
- JP1: value (none) -> thermistor
- JP6: value (none) -> Motor
- SJ1: value (none) -> vref
- SW2: value (none) -> Reset
Connections:
- net SHIELD renamed N$9
- net VIN renamed +5V
- removed net D13: R1.2, U2.PA16/I2C/I0/SERCOM1.0+3.1
- removed net N$33: D1.ANODE, F1.2
- new net LEDERROR: R8.2, U2.PA08/I2C/AIN8/SEROM0.0+2.1/I2SMCK
- new net LEDSTATUS: R1.2, U2.PA09/I2C/I9/AIN9SEROM0.1+2.0/I2SFS0
- new net N$11: LED3.A, R9.1
- new net N$12: D1.ANODE, F2.2
- new net N$3: LED2.A, R8.1
- new net VSENSE: R4.2, R7.1, U2.PA10/I107AIN110/SEROM0+2.27I2SCK
- net 3.3V: now also R9.2
- net GND: now also LED2.C, LED3.C, R7.2
- net N$36: now also F2.1; no longer F1.1
- net V+: now also R4.1
Other:
- note added: "LEDS"
- note added: "v+ Voltage"
- moved on the sheet: C1, C10, C11, C14, C15, C17, C18, C19, C2, C20, C21, C22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

Commit message: Rearange to fit old pin positions
Parts:
- removed J2: power, SparkFun-Connectors:CONN_03
- added J4: power, SparkFun-Connectors:CONN_03
- added U4: R-78E5.0-1.0, SparkFun-IC-Power:R-78E5.0-1.0
Connections:
- net +5V: now also J4.1, U4.OUT; no longer J2.2
- net GND: now also J4.2, U4.GND; no longer J2.1
- net V+: now also J4.3, U4.IN; no longer J2.3
Changed lines of the file:
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@@
 <layers>
 <layer number="1" name="Top" color="4" fill="1" visible="no" active="no"/>
+<layer number="2" name="Route2" color="1" fill="3" visible="no" active="no"/>
+<layer number="3" name="Route3" color="4" fill="3" visible="no" active="no"/>
+<layer number="4" name="Route4" color="1" fill="4" visible="no" active="no"/>
+<layer number="5" name="Route5" color="4" fill="4" visible="no" active="no"/>
+<layer number="6" name="Route6" color="1" fill="8" visible="no" active="no"/>
+<layer number="7" name="Route7" color="4" fill="8" visible="no" active="no"/>
+<layer number="8" name="Route8" color="1" fill="2" visible="no" active="no"/>
+<layer number="9" name="Route9" color="4" fill="2" visible="no" active="no"/>
+<layer number="10" name="Route10" color="1" fill="7" visible="no" active="no"/>
+<layer number="11" name="Route11" color="4" fill="7" visible="no" active="no"/>
+<layer number="12" name="Route12" color="1" fill="5" visible="no" active="no"/>
+<layer number="13" name="Route13" color="4" fill="5" visible="no" active="no"/>
+<layer number="14" name="Route14" color="1" fill="6" visible="no" active="no"/>
+<layer number="15" name="Route15" color="4" fill="6" visible="no" active="no"/>
 <layer number="16" name="Bottom" color="1" fill="1" visible="no" active="no"/>
 <layer number="17" name="Pads" color="2" fill="1" visible="no" active="no"/>
@@
 <part name="J1" library="MF_Connectors" deviceset="USB" device="_MICRO_RIGHT" value="USB"/>
 <part name="FRAME1" library="SparkFun-Aesthetics" deviceset="FRAME-LEDGER" device=""/>
-<part name="P+1" library="supply1" deviceset="V+" device=""/>
 <part name="P+2" library="supply1" deviceset="V+" device=""/>
 <part name="SUPPLY21" library="SparkFun-Aesthetics" deviceset="3.3V" device=""/>
@@
 <part name="GND15" library="supply1" deviceset="GND" device=""/>
 <part name="JP1" library="pinhead" library_urn="urn:adsk.eagle:library:325" deviceset="PINHD-1X2" device="" package3d_urn="urn:adsk.eagle:package:22435/2" value="thermistor"/>
-<part name="J2" library="SparkFun-Connectors" library_urn="urn:adsk.eagle:library:513" deviceset="CONN_03" device="" package3d_urn="urn:adsk.eagle:package:38063/1" value="power"/>
 <part name="GND16" library="supply1" deviceset="GND" device=""/>
 <part name="U2" library="atsamd51" deviceset="ATSAMD51J19" device=""/>
@@
 <part name="C1" library="swift" deviceset="CAP" device="0402" value="0.1uF"/>
 <part name="C21" library="swift" deviceset="CAP" device="0402" value="0.1uF"/>
-<part name="GND3" library="supply1" deviceset="GND" device=""/>
 <part name="SJ1" library="jumper" library_urn="urn:adsk.eagle:library:252" deviceset="SJ" device="" package3d_urn="urn:adsk.eagle:package:15471/1" value="vref"/>
 <part name="SUPPLY5" library="SparkFun-Aesthetics" deviceset="3.3V" device=""/>
@@
 <part name="P+6" library="supply1" library_urn="urn:adsk.eagle:library:371" deviceset="+5V" device=""/>
 <part name="F2" library="adafruit" deviceset="PTCFUSE" device="-1206" value="500mA"/>
+<part name="J4" library="SparkFun-Connectors" library_urn="urn:adsk.eagle:library:513" deviceset="CONN_03" device="" package3d_urn="urn:adsk.eagle:package:38063/1" value="power"/>
+<part name="P+8" library="supply1" deviceset="V+" device=""/>
+<part name="GND24" library="supply1" deviceset="GND" device=""/>
+<part name="P+9" library="supply1" library_urn="urn:adsk.eagle:library:371" deviceset="+5V" device=""/>
+<part name="U4" library="SparkFun-IC-Power" library_urn="urn:adsk.eagle:library:526" deviceset="R-78E5.0-1.0" device="" package3d_urn="urn:adsk.eagle:package:39086/1"/>
+<part name="GND3" library="supply1" deviceset="GND" device=""/>
+<part name="P+1" library="supply1" deviceset="V+" device=""/>
 <part name="P+7" library="supply1" library_urn="urn:adsk.eagle:library:371" deviceset="+5V" device=""/>
 </parts>
@@
 <instance part="J1" gate="G$1" x="7.62" y="45.72"/>
 <instance part="FRAME1" gate="G$2" x="332.74" y="2.54"/>
-<instance part="P+1" gate="1" x="274.32" y="58.42" smashed="yes" rot="MR0">
-<attribute name="VALUE" x="274.32" y="60.96" size="1.778" layer="96" rot="MR0"/>
-</instance>
 <instance part="P+2" gate="1" x="124.46" y="134.62" smashed="yes">
 <attribute name="VALUE" x="124.46" y="137.16" size="1.778" layer="96" rot="MR0"/>
@@
 <instance part="GND15" gate="1" x="421.64" y="162.56"/>
 <instance part="JP1" gate="G$1" x="396.24" y="182.88" rot="R180"/>
-<instance part="J2" gate="J$1" x="259.08" y="48.26"/>
 <instance part="GND16" gate="1" x="104.14" y="93.98"/>
 <instance part="U2" gate="G$1" x="139.7" y="261.62"/>
@@
 <attribute name="VALUE" x="75.184" y="279.781" size="1.778" layer="96"/>
 </instance>
-<instance part="GND3" gate="1" x="274.32" y="38.1"/>
 <instance part="SJ1" gate="1" x="317.5" y="287.02"/>
 <instance part="SUPPLY5" gate="G$1" x="304.8" y="294.64"/>
@@
 <instance part="P+6" gate="1" x="373.38" y="144.78"/>
 <instance part="F2" gate="G$1" x="53.34" y="48.26"/>
-<instance part="P+7" gate="1" x="279.4" y="58.42"/>
+<instance part="J4" gate="J$1" x="261.62" y="20.32"/>
+<instance part="P+8" gate="1" x="284.48" y="30.48" smashed="yes" rot="MR0">
+<attribute name="VALUE" x="284.48" y="33.02" size="1.778" layer="96" rot="MR0"/>
+</instance>
+<instance part="GND24" gate="1" x="284.48" y="10.16"/>
+<instance part="P+9" gate="1" x="289.56" y="30.48"/>
+<instance part="U4" gate="G$1" x="180.34" y="17.78"/>
+<instance part="GND3" gate="1" x="180.34" y="0" smashed="yes">
+<attribute name="VALUE" x="177.8" y="-2.54" size="1.778" layer="96"/>
+</instance>
+<instance part="P+1" gate="1" x="162.56" y="22.86" smashed="yes" rot="MR0">
+<attribute name="VALUE" x="162.56" y="25.4" size="1.778" layer="96" rot="MR0"/>
+</instance>
+<instance part="P+7" gate="1" x="203.2" y="22.86"/>
 </instances>
 <busses>
@@
 </segment>
 <segment>
-<pinref part="J2" gate="J$1" pin="1"/>
-<wire x1="266.7" y1="45.72" x2="274.32" y2="45.72" width="0.1524" layer="91"/>
-<pinref part="GND3" gate="1" pin="GND"/>
-<wire x1="274.32" y1="45.72" x2="274.32" y2="40.64" width="0.1524" layer="91"/>
-</segment>
-<segment>
 <pinref part="GND17" gate="1" pin="GND"/>
 <pinref part="C22" gate="G$1" pin="2"/>
@@
 <pinref part="R7" gate="G$1" pin="2"/>
 <wire x1="340.36" y1="165.1" x2="340.36" y2="172.72" width="0.1524" layer="91"/>
+</segment>
+<segment>
+<pinref part="GND24" gate="1" pin="GND"/>
+<wire x1="284.48" y1="20.32" x2="284.48" y2="12.7" width="0.1524" layer="91"/>
+<pinref part="J4" gate="J$1" pin="2"/>
+<wire x1="269.24" y1="20.32" x2="284.48" y2="20.32" width="0.1524" layer="91"/>
+</segment>
+<segment>
+<pinref part="U4" gate="G$1" pin="GND"/>
+<pinref part="GND3" gate="1" pin="GND"/>
+<wire x1="180.34" y1="10.16" x2="180.34" y2="2.54" width="0.1524" layer="91"/>
 </segment>
 </net>
@@
 <net name="V+" class="0">
 <segment>
-<pinref part="P+1" gate="1" pin="V+"/>
-<wire x1="274.32" y1="55.88" x2="274.32" y2="50.8" width="0.1524" layer="91"/>
-<wire x1="274.32" y1="50.8" x2="266.7" y2="50.8" width="0.1524" layer="91"/>
-<pinref part="J2" gate="J$1" pin="3"/>
-</segment>
-<segment>
 <pinref part="U$1" gate="G$1" pin="VBB"/>
 <wire x1="121.92" y1="124.46" x2="124.46" y2="124.46" width="0.1524" layer="91"/>
@@
 <pinref part="R4" gate="G$1" pin="1"/>
 <wire x1="340.36" y1="208.28" x2="340.36" y2="203.2" width="0.1524" layer="91"/>
+</segment>
+<segment>
+<pinref part="P+8" gate="1" pin="V+"/>
+<wire x1="284.48" y1="27.94" x2="284.48" y2="22.86" width="0.1524" layer="91"/>
+<pinref part="J4" gate="J$1" pin="3"/>
+<wire x1="269.24" y1="22.86" x2="284.48" y2="22.86" width="0.1524" layer="91"/>
+</segment>
+<segment>
+<pinref part="P+1" gate="1" pin="V+"/>
+<wire x1="162.56" y1="20.32" x2="162.56" y2="17.78" width="0.1524" layer="91"/>
+<pinref part="U4" gate="G$1" pin="IN"/>
+<wire x1="162.56" y1="17.78" x2="172.72" y2="17.78" width="0.1524" layer="91"/>
 </segment>
 </net>
@@
 </segment>
 <segment>
-<wire x1="266.7" y1="48.26" x2="279.4" y2="48.26" width="0.1524" layer="91"/>
-<pinref part="J2" gate="J$1" pin="2"/>
-<wire x1="279.4" y1="48.26" x2="279.4" y2="55.88" width="0.1524" layer="91"/>
+<wire x1="289.56" y1="17.78" x2="289.56" y2="27.94" width="0.1524" layer="91"/>
+<pinref part="P+9" gate="1" pin="+5V"/>
+<pinref part="J4" gate="J$1" pin="1"/>
+<wire x1="269.24" y1="17.78" x2="289.56" y2="17.78" width="0.1524" layer="91"/>
+</segment>
+<segment>
+<pinref part="U4" gate="G$1" pin="OUT"/>
 <pinref part="P+7" gate="1" pin="+5V"/>
-</segment>
-</net>
+<wire x1="187.96" y1="17.78" x2="203.2" y2="17.78" width="0.1524" layer="91"/>
+<wire x1="203.2" y1="17.78" x2="203.2" y2="20.32" width="0.1524" layer="91"/>
+</segment>
+</net>
