File: MEchaduino_03.brd (EAGLE design)
At the start: 41.9 x 41.9 mm, 56 parts, among them J1 USB, J3 signals, J4 power, SW2 Reset, U1 TLV70233PDBVR, U2 ATSAMD51J19, U3 TXB0104, U4 R-78E5.0-1.0, Y1 3.2768KHZ

Commit message: Finalized version of PCB for manufacturing
Parts:
- removed C17: 22pF, swift:0603-CAP
- removed C19: 1.0uF, swift:0402-CAP
- removed D2: 20V-1A, Seeed-Diode:SOD-123
- removed D4: RED, SparkFun-LED:LED-0603
- removed D5: Yellow, SparkFun-LED:LED-0603
- removed F2: 500mA, adafruit:R1206
- removed J4: power, SparkFun-Connectors:1X03
- removed JP1: thermistor, pinhead:1X02
- removed JP6: Motor, SparkFun-Connectors:1X04
- removed L3: 2500R-50MA, Seeed-Inductor:L0603
- removed R12, R13: .15 Ohm 1%, adafruit:R1206
- removed SW2: Reset, MF_Switches:TACT4.2MM
- removed U3: TXB0104, SparkFun-IC-Comms:TSSOP14
- added C23: 100nf, Seeed-Capacitor:C0402
- added CN1: 3p-2.54, Seeed-Connector:H3-2.54
- added CT1: 47UF, Seeed-Capacitor:ELECTRO-SMD-C-6MM
- added D1, D6: YELLOW-0603, Seeed-LED:LED-0603
- added D7: GREEN-0603, Seeed-LED:LED-0603
- added F1: SMD1206R500SF, Seeed-Fuse:F1206
- added J2: 2p-2.54, Seeed-Connector:H2-2.54
- added L2: 10UH-225MA, Seeed-Inductor:L0806
- added R10: 6.8K, Seeed-Resistor:R0603
- added R11: 330R, Seeed-Resistor:R0402
- added SW3: DHT-4235A, Seeed-Switch:SW4-SMD-4.2X3.2X2.5MM
- added U$4: MECHADUINO_LOGO, stepper_servo_prototype_1:MECHADUINO_LOGO
- added U6: XC6204B332MR-SOT23-5, Seeed-IC:SOT-23-5
- added USB2: ZX62-B-5PA, Seeed-Connector:MICRO-USB5+6P-SMD-0.65-AB
- C1, C10, C14, C15, C18, C2, C20, C21, C22, C4, C5, C8: value 0.1uF -> 100nf; device swift:0402-CAP -> Seeed-Capacitor:C0402
- C11: value 1uF -> 100nf; device swift:0402-CAP -> Seeed-Capacitor:C0402
- C12: value 100uF -> 100nf; device SparkFun-Capacitors:PANASONIC_D -> Seeed-Capacitor:C0402
- C13: value 1.0uF -> 100nf; device swift:0603-CAP -> Seeed-Capacitor:C0603
- C16, C7: value 0.1uF -> 27pf; device swift:0402-CAP -> Seeed-Capacitor:C0402
- C3: value 22pF -> 10nf; device swift:0603-CAP -> Seeed-Capacitor:C0603
- C6: value 0.01uF -> 1UF 6.3V; device swift:0603-CAP -> Seeed-Capacitor:C0402
- C9: value 1.0uF -> 1UF 6.3V; device swift:0402-CAP -> Seeed-Capacitor:C0402
- D3: value GREEN -> 20V-500MA; device SparkFun-LED:LED-0603 -> Seeed-Diode:SOD-123
- J1: value USB -> 4p-2.54; device MF_Connectors:MICROUSB-RIGHT -> Seeed-Connector:H4-2.54
- R1, R8: value 1k -> 330R; device rcl:R0402 -> Seeed-Resistor:R0402
- R2: value 10k -> 10K 1/16W; device rcl:R0402 -> Seeed-Resistor:R0402
- R3: value 10k -> 100K; device rcl:R0402 -> Seeed-Resistor:R0402
- R4, R5: value 100k -> 10K 1/16W; device rcl:R0402 -> Seeed-Resistor:R0402
- R6: value 10k -> R150, 3/4W, 1%; device rcl:R0402 -> adafruit:R1206
- R7: value 6k8 -> R150, 3/4W, 1%; device rcl:R0402 -> adafruit:R1206
- R9: value 1k -> 100K; device rcl:R0402 -> Seeed-Resistor:R0402
- U1: value TLV70233PDBVR -> TXS0108EPWR-TSSOP20; device MF_IC_Power:SOT-23-5 -> Seeed-IC:TSSOP20-0.65-6.5X4.4MM
- moved C3 31.4 mm to (31.8, 7.87), turned to 0 degrees
- moved R6 27.9 mm to (31.4, 4.06), turned to 0 degrees
- moved C22 26.5 mm to (6.22, 23.7), turned to 90 degrees
- moved R7 24.3 mm to (23.7, 4.06), turned to 180 degrees
- moved C16 22.6 mm to (24.8, 38.7), turned to 135 degrees
- moved C12 22.2 mm to (19.1, 31.8), flipped to the bottom, turned to 90 degrees
- moved J1 21.7 mm to (27.6, 1.52), turned to 270 degrees
- moved C6 21.0 mm to (14.6, 20.1), turned to 180 degrees
- moved R2 21.0 mm to (35.4, 31.5), turned to 135 degrees
- moved C20 19.8 mm to (26.9, 39.6), turned to 90 degrees
- moved C8 15.3 mm to (19.9, 16.9), flipped to the bottom, turned to 270 degrees
- moved U1 14.4 mm to (14.5, 33.8), flipped to the bottom, turned to 0 degrees
- moved C21 13.5 mm to (17.8, 22.2), flipped to the top, turned to 225 degrees
- moved R9 10.7 mm to (13.2, 25.4)
- moved D3 10.5 mm to (13.5, 16.5), turned to 0 degrees
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Connections:
- removed net N$36: F2.1, J1.1
- new net N$17: J3.P$5, U1.18
- new net SHIELD: L1.1, USB2.P1, USB2.P2, USB2.P3, USB2.P4, USB2.P5, USB2.P6
- new net VBUS: F1.1, USB2.1
- net +5V: now also C4.2, C6.2, CN1.1, D3.-, U1.19, U6.1, U6.3; no longer C4.1, C9.1, D2.-, J4.1, U1.P$1, U1.P$3, U3.14
- net 3.3V: now also C10.2, C12.2, C14.2, C18.2, C2.2, C21.2, C8.2, C9.2, R11.2, R3.1, R4.2, U1.2, U6.5; no longer C10.1, C14.1, C16.1, C18.1, C19.1, C2.1, C20.1, C7.1, R5.1, R6.1, R9.2, U1.P$5, U3.1
- net ARDUINO_D0: now also U1.4; no longer U3.2
- net ARDUINO_D1: now also U1.5; no longer U3.3
- net ARDUINO_D2: now also U1.6; no longer U3.4
- net ARDUINO_D3: now also U1.7; no longer U3.5
- net AREF: now also C20.2; no longer C22.1
- net CRYST1: now also C16.2; no longer C3.2
- net CRYST2: now also C7.2; no longer C17.2
- net D+: now also USB2.3; no longer J1.3
- net D-: now also USB2.2; no longer J1.2
- net GND: now also C1.1, C10.1, C12.1, C13.1, C14.1, C16.1, C18.1, C2.1, C20.1, C21.1, C22.1, C23.1, C4.1, C5.1, C6.1, C7.1, C8.1, C9.1, CN1.2, CT1.-, D1.-, D6.-, D7.-, J2.1, L1.2, R10.1, R6.2, SW3.3, U1.11, U6.2, USB2.5; no longer C1.2, C10.2, C12.-, C13.2, C14.2, C16.2, C17.1, C18.2, C19.2, C2.2, C20.2, C21.2, C22.2, C4.2, C5.2, C6.2, C7.2, C8.2, C9.2, D3.C, D4.C, D5.C, J1.5, J4.2, JP1.1, L3.2, R12.2, R13.2, SW2.P$3, SW2.P$4, U1.P$2, U3.7
- net I_SENSE_COIL_A: now also R7.1; no longer R13.1
- net I_SENSE_COIL_B: now also R6.1; no longer R12.1
- net LEDERROR: now also R1.2; no longer R8.2
- net LEDSTATUS: now also R8.2; no longer R1.2
- net N$1: now also D6.+, R8.1; no longer D5.A, R1.1
- net N$10: now also L2.2; no longer L1.2
- net N$11: now also D7.+, R11.1; no longer D3.A, R9.1
- net N$12: now also D3.+, F1.2; no longer D2.+, F2.2
- net N$13: now also J1.1; no longer JP6.4
- net N$14: now also J1.4; no longer JP6.1
- net N$15: now also J1.3; no longer JP6.2
- net N$16: now also J1.2; no longer JP6.3
- net N$2: now also U1.17; no longer U3.13
- net N$23: now also J2.2, R5.1; no longer JP1.2, R5.2
- net N$3: now also D1.+, R1.1; no longer D4.A, R8.1
- net N$4: now also U1.16; no longer U3.12
- net N$5: now also U1.15; no longer U3.11
- net N$6: now also R4.1, U1.10; no longer R2.1, U3.8
- net N$7: now also U1.14; no longer U3.10
- net N$8: now also C1.2, C23.2, C5.2, L2.1; no longer C1.1, C21.1, C5.1, L1.1
- net N$9: now also J3.P$6, U1.20; no longer J1.S1, J1.S2, J1.S3, J1.S4, J1.S5, J1.S6, J1.S7, J1.S8, L3.1
- net RESET: now also R2.1, SW3.1; no longer R6.2, SW2.P$1, SW2.P$2
- net SCL: now also U1.1; no longer J3.P$5
- net SDA: now also U1.3; no longer J3.P$6
- net TH1: now also C22.2, R5.2; no longer C8.1, R3.1
- net V+: now also C13.2, C3.2, CN1.3, CT1.+, R9.2; no longer C12.+, C13.1, C6.1, J4.3, R4.1
- net VSENSE: now also R10.2, R9.1; no longer R4.2, R7.1
Routing:
- net GND: track 125.7 -> 109.1 mm, vias 26 -> 24
- net SHIELD: track 0.00 -> 15.8 mm
- net N$17: track 0.00 -> 6.74 mm
- net SDA: track 11.0 -> 15.9 mm
- net N$9: track 12.3 -> 7.71 mm
- net N$36: track 3.80 -> 0.00 mm
- net RESET: track 9.99 -> 7.02 mm
- net 3.3V: track 114.6 -> 117.4 mm, vias 7 -> 5
- net VBUS: track 0.00 -> 2.70 mm
- net N$12: track 22.1 -> 24.6 mm
- net N$5: track 7.24 -> 5.23 mm
- net ARDUINO_D1: track 20.0 -> 22.0 mm
- net ARDUINO_D0: track 19.7 -> 21.5 mm
- net N$6: track 3.10 -> 1.32 mm, vias 1 -> 0
- net ARDUINO_D3: track 21.1 -> 22.7 mm
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