File: MEchaduino_03.sch (EAGLE design)
At the start: 56 parts, among them J1 USB, J3 signals, J4 power, SW2 Reset, U1 TLV70233PDBVR, U2 ATSAMD51J19, U3 TXB0104, U4 R-78E5.0-1.0, Y1 3.2768KHZ

Commit message: Finalized version of PCB for manufacturing
Parts:
- removed C17: 22pF, swift:CAP0603
- removed C19: 1.0uF, swift:CAP0402
- removed D2: 20V-1A, Seeed-Diode:SMD-DIODE-SCHOTTKY-20V-1A(SOD-123)
- removed D4: RED, SparkFun-LED:LED-RED0603
- removed D5: Yellow, SparkFun-LED:LED-YELLOW0603
- removed F2: 500mA, adafruit:PTCFUSE-1206
- removed J4: power, SparkFun-Connectors:CONN_03
- removed JP1: thermistor, pinhead:PINHD-1X2
- removed JP6: Motor, SparkFun-Connectors:M04PTH
- removed L3: 2500R-50MA, Seeed-Inductor:SMD-FERRITE-BEAD-2500R-50MA(0603)
- removed R12, R13: .15 Ohm 1%, adafruit:R-US_R1206
- removed SW2: Reset, MF_Switches:TACT_4.2MM
- removed U3: TXB0104, SparkFun-IC-Comms:TXB0104PWR
- added C23: 100nf, Seeed-Capacitor:CERAMIC-100NF-25V-10%-X7R(0402)
- added CN1: 3p-2.54, Seeed-Connector:DIP-BLACK-MALE-HEADER-VERT(3P-2.54)
- added CT1: 47UF, Seeed-Capacitor:ALUMINUM-SMD-47UF-25V(D6.3-H5.3MM)
- added D1, D6: YELLOW-0603, Seeed-LED:SMD-LED-CLEAR-YELLOW(0603)
- added D7: GREEN-0603, Seeed-LED:SMD-LED-CLEAR-GREEN(0603)
- added F1: SMD1206R500SF, Seeed-Fuse:SMD-PPTC-500MA(1206)
- added J2: 2p-2.54, Seeed-Connector:DIP-BLACK-MALE-HEADER-VERT(2P-2.54)
- added L2: 10UH-225MA, Seeed-Inductor:SMD-INDUCTOR-10UH-225MA-10%(0806)
- added R10: 6.8K, Seeed-Resistor:SMD-RES-6.8K-1%-1/10W(0603)
- added R11: 330R, Seeed-Resistor:SMD-RES-330R-1%-1/16W(0402)
- added SW3: DHT-4235A, Seeed-Switch:SMD-BUTTON-TOP-DHT-4235A(4P-4.2X3.2MM)
- added U$4: MECHADUINO_LOGO, stepper_servo_prototype_1:MECHADUINO_LOGO
- added U6: XC6204B332MR-SOT23-5, Seeed-IC:PMIC-LDO-XC6204B332MR(SOT23-5)
- added USB2: ZX62-B-5PA, Seeed-Connector:MICRO-USB-SMD(ZX62-B-5PA)
- C1, C10, C14, C15, C18, C2, C20, C21, C22, C4, C5, C8: value 0.1uF -> 100nf; device swift:CAP0402 -> Seeed-Capacitor:CERAMIC-100NF-25V-10%-X7R(0402)
- C11: value 1uF -> 100nf; device swift:CAP0402 -> Seeed-Capacitor:CERAMIC-100NF-25V-10%-X7R(0402)
- C12: value 100uF -> 100nf; device SparkFun-Capacitors:CAP_POLD -> Seeed-Capacitor:CERAMIC-100NF-25V-10%-X7R(0402)
- C13: value 1.0uF -> 100nf; device swift:CAP0603 -> Seeed-Capacitor:CERAMIC-100NF-50V-10%-X7R(0603)
- C16, C7: value 0.1uF -> 27pf; device swift:CAP0402 -> Seeed-Capacitor:CERAMIC-27PF-50V-5%-NPO(0402)
- C3: value 22pF -> 10nf; device swift:CAP0603 -> Seeed-Capacitor:CERAMIC-10NF-50V-10%-X7R(0603)
- C6: value 0.01uF -> 1UF 6.3V; device swift:CAP0603 -> Seeed-Capacitor:CERAMIC-1UF-6.3V-10%-X5R(0402)
- C9: value 1.0uF -> 1UF 6.3V; device swift:CAP0402 -> Seeed-Capacitor:CERAMIC-1UF-6.3V-10%-X5R(0402)
- D3: value GREEN -> 20V-500MA; device SparkFun-LED:LED-GREEN0603 -> Seeed-Diode:SMD-DIODE-SCHOTTKY-20V-500MA(SOD-123)
- J1: value USB -> 4p-2.54; device MF_Connectors:USB_MICRO_RIGHT -> Seeed-Connector:DIP-BLACK-MALE-HEADER-VERT(4P-2.54)
- J3: LABEL00 *D3 -> D3; LABEL01 *D2 -> D2; LABEL02 *D1 -> D1; LABEL03 *D0 -> D0; LABEL04 SCL -> SDA; LABEL05 SDA -> SCL
- R1, R8: value 1k -> 330R; device rcl:R-US_R0402 -> Seeed-Resistor:SMD-RES-330R-1%-1/16W(0402)
- R2: value 10k -> 10K 1/16W; device rcl:R-US_R0402 -> Seeed-Resistor:SMD-RES-10K-1%-1/16W(0402)
- R3: value 10k -> 100K; device rcl:R-US_R0402 -> Seeed-Resistor:SMD-RES-100K-1%-1/16W(0402)
- R4, R5: value 100k -> 10K 1/16W; device rcl:R-US_R0402 -> Seeed-Resistor:SMD-RES-10K-1%-1/16W(0402)
- R6: value 10k -> R150, 3/4W, 1%; device rcl:R-US_R0402 -> adafruit:R-US_R1206; MPN (none) -> KRL1632E-M-R150-F-T5
- R7: value 6k8 -> R150, 3/4W, 1%; device rcl:R-US_R0402 -> adafruit:R-US_R1206; MPN (none) -> KRL1632E-M-R150-F-T5
- R9: value 1k -> 100K; device rcl:R-US_R0402 -> Seeed-Resistor:SMD-RES-100K-1%-1/16W(0402)
- U$1: MPN (none) -> AS5047D-ATSM
- U$3: MPN (none) -> A4953ELJTR-T
- U1: value TLV70233PDBVR -> TXS0108EPWR-TSSOP20; device MF_IC_Power:TLV70233PDBVR -> Seeed-IC:LOGIC-TXS0108EPWR(TSSOP20)
- U2: MPN (none) -> ATSAMD51J19A-AU
Connections:
- removed net N$36: F2.1, J1.5V
- new net N$17: J3.PIN4, U1.B2
- new net SHIELD: L1.1, USB2.SHIELD
- new net VBUS: F1.1, USB2.VBUS
- net +5V: now also C4.2, C6.2, CN1.P$1, D3.-, U1.VCCB, U6.CE, U6.VIN; no longer C4.1, C9.1, D2.-, J4.1, U1.EN, U1.VIN, U3.VCCB
- net 3.3V: now also C10.2, C12.2, C14.2, C18.2, C2.2, C21.2, C8.2, C9.2, R11.2, R3.1, R4.2, U1.VCCA, U6.VOUT; no longer C10.1, C14.1, C16.1, C18.1, C19.1, C2.1, C20.1, C7.1, R5.1, R6.1, R9.2, U1.VOUT, U3.VCCA
- net ARDUINO_D0: now also U1.A3; no longer U3.A1
- net ARDUINO_D1: now also U1.A4; no longer U3.A2
- net ARDUINO_D2: now also U1.A5; no longer U3.A3
- net ARDUINO_D3: now also U1.A6; no longer U3.A4
- net AREF: now also C20.2; no longer C22.1
- net CRYST1: now also C16.2; no longer C3.2
- net CRYST2: now also C7.2; no longer C17.2
- net D+: now also USB2.D+; no longer J1.D+
- net D-: now also USB2.D-; no longer J1.D-
- net GND: now also C1.1, C10.1, C12.1, C13.1, C14.1, C16.1, C18.1, C2.1, C20.1, C21.1, C22.1, C23.1, C4.1, C5.1, C6.1, C7.1, C8.1, C9.1, CN1.P$2, CT1.-, D1.-, D6.-, D7.-, J2.1, L1.2, R10.1, R6.2, SW3.B0, U1.GND, U6.VSS, USB2.GND; no longer C1.2, C10.2, C12.-, C13.2, C14.2, C16.2, C17.1, C18.2, C19.2, C2.2, C20.2, C21.2, C22.2, C4.2, C5.2, C6.2, C7.2, C8.2, C9.2, D3.C, D4.C, D5.C, J1.GND, J4.2, JP1.1, L3.2, R12.2, R13.2, SW2.P$3, SW2.P$4, U1.GND/ADJ, U3.GND
- net I_SENSE_COIL_A: now also R7.1; no longer R13.1
- net I_SENSE_COIL_B: now also R6.1; no longer R12.1
- net LEDERROR: now also R1.2; no longer R8.2
- net LEDSTATUS: now also R8.2; no longer R1.2
- net N$1: now also D6.+, R8.1; no longer D5.A, R1.1
- net N$10: now also L2.2; no longer L1.2
- net N$11: now also D7.+, R11.1; no longer D3.A, R9.1
- net N$12: now also D3.+, F1.2; no longer D2.+, F2.2
- net N$13: now also J1.P$1; no longer JP6.4
- net N$14: now also J1.P$4; no longer JP6.1
- net N$15: now also J1.P$3; no longer JP6.2
- net N$16: now also J1.P$2; no longer JP6.3
- net N$2: now also U1.B3; no longer U3.B1
- net N$23: now also J2.2, R5.1; no longer JP1.2, R5.2
- net N$3: now also D1.+, R1.1; no longer D4.A, R8.1
- net N$4: now also U1.B4; no longer U3.B2
- net N$5: now also U1.B5; no longer U3.B3
- net N$6: now also R4.1, U1.OE; no longer R2.1, U3.OE
- net N$7: now also U1.B6; no longer U3.B4
- net N$8: now also C1.2, C23.2, C5.2, L2.1; no longer C1.1, C21.1, C5.1, L1.1
- net N$9: now also J3.PIN5, U1.B1; no longer J1.SLD, L3.1
- net RESET: now also R2.1, SW3.A0; no longer R6.2, SW2.P$1, SW2.P$2
- net SCL: now also U1.A1; no longer J3.PIN4
- net SDA: now also U1.A2; no longer J3.PIN5
- net TH1: now also C22.2, R5.2; no longer C8.1, R3.1
- net V+: now also C13.2, C3.2, CN1.P$3, CT1.+, R9.2; no longer C12.+, C13.1, C6.1, J4.3, R4.1
- net VSENSE: now also R10.2, R9.1; no longer R4.2, R7.1
Other:
- note removed: "TLV70233PDBVR ---------------- Iout (max): 300mA Vin (max): 6.0V Vdo (typ): 220mV Iq: 35uA"
- moved on the sheet: L1, R6, R7
